Commit message: Add a dummy link to base_link

File: urdf/dd_bot.urdf (robot description, URDF)
Before this commit: robot dd_bot, 5 links, 4 joints
Links:
- added link base_link_parent
Joints:
- added joint paret_base_link: type fixed, parent base_link_parent, child base_link, origin xyz=0 0 0 rpy=0 0 0
